Commit message: Phase 2: cgo + RDK API alignment, URDF cleanup
cgo arm package builds clean against libfranka 0.9.2 headers; go vet
clean across whole module. URDF parses to a 7-DoF model.

Co-Authored-By: Claude Opus 4.7 (1M context) <noreply@anthropic.com>

File: arm/panda_arm.urdf (robot description, URDF)
Before this commit: robot panda, 11 links, 10 joints
Links:
- link panda_link0: mass 0.629769273993887 -> None; geometry 
- link panda_link1: mass 4.970684 -> None; geometry 
- link panda_link2: mass 0.646926 -> None; geometry 
- link panda_link3: mass 3.228604 -> None; geometry 
- link panda_link4: mass 3.587895 -> None; geometry 
- link panda_link5: mass 1.225946 -> None; geometry 
- link panda_link6: mass 1.666555 -> None; geometry 
- link panda_link7: mass 7.35522e-01 -> None; geometry 
- link panda_link8: mass 1e-10 -> None
- link panda_mount: geometry 
