Commit message: Render Franka arm in 3D Scene, add STL files, improve Makefile multi-arch docker build
Signed-off-by: John Walicki <johnwalicki@gmail.com>

File: arm/panda_arm.urdf (robot description, URDF)
Before this commit: robot panda, 11 links, 10 joints
Links:
- link panda_link0: geometry collision mesh filename=meshes/panda/link0.stl
- link panda_link1: geometry collision mesh filename=meshes/panda/link1.stl
- link panda_link2: geometry collision mesh filename=meshes/panda/link2.stl
- link panda_link3: geometry collision mesh filename=meshes/panda/link3.stl
- link panda_link4: geometry collision mesh filename=meshes/panda/link4.stl
- link panda_link5: geometry collision mesh filename=meshes/panda/link5.stl
- link panda_link6: geometry collision mesh filename=meshes/panda/link6.stl
- link panda_link7: geometry collision mesh filename=meshes/panda/link7.stl
